File: project/pcb/attiny85_timer/attiny85_timer.kicad_pcb (KiCad board)
At the start: 2 copper layers, 50 x 50 mm, 25 parts, among them J1 USB-C, J2 AVR-ISP, J3 AUX_OUT, U1 NE555D, U2 ATtiny85-20SU

Commit message: fix(pcb): audit and resolve connector orientations and edge clearances across all boards
- Fix J1/J2 audio jack orientations on tht_opamp_eq from 270 deg (inward) to 90 deg (facing outward off South edge)
- Fix J1 USB-C receptacle alignment on attiny85_timer to sit flush with West board edge (shifted from X=6.5mm to X=4.3mm)
- Refine placement_validator to distinguish vertical through-hole pin headers from horizontal directional headers
- Resolve remaining DRC track crossings and thermal starvations on tht_opamp_eq (0 DRC, 0 unconnected items)
- Re-export complete manufacturing packages (Gerbers, drills, BOM, CPL, 3D renders) for attiny85_timer and tht_opamp_eq
- Verify 23/23 tests pass across test suite

Co-authored-by: Mema <mema@glassgallery.my.id>
Parts:
- moved J1 2.20 mm to (4.30, 25.0)
Routing:
- net +5V: track 158.3 -> 162.7 mm
- net CC2: track 2.54 -> 4.74 mm
- net CC1: track 2.54 -> 4.74 mm
Changed lines of the file:
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@@
 	(footprint "USB_C_Receptacle_HRO_TYPE-C-31-M-12"
 		(layer "F.Cu")
-		(at 6.5 25 -90)
+		(at 4.3 25 -90)
 		(descr "USB Type-C receptacle for USB 2.0 and PD, http://www.krhro.com/uploads/soft/180320/1-1P320120243.pdf")
 		(tags "usb usb-c 2.0 pd")
@@
 	)
 	(segment
-		(start 10.545 28.25)
-		(end 9.63 29.32)
+		(start 8.345 28.25)
+		(end 7.43 29.32)
 		(width 0.25)
 		(layer "F.Cu")
@@
 	)
 	(segment
-		(start 10.545 21.75)
-		(end 9.63 20.68)
+		(start 8.345 21.75)
+		(end 7.43 20.68)
 		(width 0.25)
 		(layer "F.Cu")
@@
 	)
 	(segment
-		(start 10.545 22.55)
+		(start 8.345 22.55)
 		(end 11.8 22.55)
 		(width 0.35)
@@
 	)
 	(segment
-		(start 10.545 27.45)
+		(start 8.345 27.45)
 		(end 11.8 27.45)
 		(width 0.35)
@@
 	)
 	(segment
-		(start 10.545 23.75)
+		(start 8.345 23.75)
 		(end 13.088 23.75)
 		(width 0.25)
@@
 	)
 	(segment
-		(start 10.545 26.75)
+		(start 8.345 26.75)
 		(end 13.088 26.75)
 		(width 0.25)
