File: project/pcb/tht_opamp_eq/tht_opamp_eq.kicad_pcb (KiCad board)
At the start: 2 copper layers, 88 x 61 mm, 51 parts, among them J1 AUDIO_IN, J2 AUDIO_OUT, J3 BAT_3V3, U1 MCP6004

Commit message: fix(pcb): audit and resolve connector orientations and edge clearances across all boards
- Fix J1/J2 audio jack orientations on tht_opamp_eq from 270 deg (inward) to 90 deg (facing outward off South edge)
- Fix J1 USB-C receptacle alignment on attiny85_timer to sit flush with West board edge (shifted from X=6.5mm to X=4.3mm)
- Refine placement_validator to distinguish vertical through-hole pin headers from horizontal directional headers
- Resolve remaining DRC track crossings and thermal starvations on tht_opamp_eq (0 DRC, 0 unconnected items)
- Re-export complete manufacturing packages (Gerbers, drills, BOM, CPL, 3D renders) for attiny85_timer and tht_opamp_eq
- Verify 23/23 tests pass across test suite

Co-authored-by: Mema <mema@glassgallery.my.id>
Parts:
- moved J1 6.00 mm to (20.0, 50.0), turned to 90 degrees
- moved J2 6.00 mm to (74.0, 50.0), turned to 90 degrees
Routing:
- net IN_R_RAW: track 58.1 -> 90.0 mm, vias 0 -> 2
- net OUT_L_JACK: track 98.1 -> 111.5 mm
- net GND: track 11.1 -> 22.2 mm
- net OUT_R_JACK: track 42.1 -> 34.7 mm, vias 0 -> 1
- net IN_L_RAW: track 20.2 -> 21.9 mm
